File: morpho64_shield/power.kicad_sch (KiCad schematic)
At the start: 14 parts, among them J4 Screw_Terminal_01x03, U4 AP63203WU

Commit message: First part of layout
Parts:
- C10, C11, C7: footprint (none) -> Capacitor_SMD:C_0603_1608Metric
- C3, C4: footprint (none) -> Capacitor_SMD:C_1206_3216Metric
- C5, C6: footprint (none) -> Capacitor_SMD:CP_Elec_16x17.5
- C8, C9: footprint (none) -> Capacitor_SMD:C_0805_2012Metric
- J4: footprint (none) -> TerminalBlock_4Ucon:TerminalBlock_4Ucon_1x03_P3.50mm_Vertical
- L1: footprint (none) -> Inductor_SMD:L_7.3x7.3_H4.5
- NT1: footprint (none) -> NetTie:NetTie-2_SMD_Pad0.5mm
Connections:
- net +3V3: now also L1.1; no longer L1.2
- net at C7.2, U4.5 (SW): now also L1.2; no longer L1.1
Other:
- note added: "Přidat nějaké ochrané diody pro případ odpojení napájení"
- moved on the sheet: L1

Commit message: First PCB order
Parts:
- C5, C6: footprint Capacitor_SMD:CP_Elec_16x17.5 -> Capacitor_SMD:CP_Elec_10x7.7
Connections:
- net SW: now reaches C7.2, L1.2, U4.5 (SW)
Changed lines of the file:
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@@
+		)
+	)
+	(label "SW"
+		(at 199.39 36.83 0)
+		(effects
+			(font
+				(size 1.27 1.27)
+			)
+			(justify left bottom)
 		)
 	)
@@
 			)
 		)
-		(property "Footprint" "Capacitor_SMD:CP_Elec_16x17.5"
+		(property "Footprint" "Capacitor_SMD:CP_Elec_10x7.7"
 			(at 88.5952 49.53 0)
 			(hide yes)
@@
 			)
 		)
-		(property "Footprint" "Capacitor_SMD:CP_Elec_16x17.5"
+		(property "Footprint" "Capacitor_SMD:CP_Elec_10x7.7"
 			(at 88.5952 59.69 0)
 			(hide yes)
